Commit message: update rfl using new compas_robot

File: src/compas_fab/data/robot_library/rfl/urdf/robot_description.urdf (robot description, URDF)
Before this commit: robot rfl, 44 links, 43 joints
Links:
- link bridge1: mass 120.00000 -> 120.0
- link bridge2: mass 120.00000 -> 120.0
- link robot11_base: mass 120.00000 -> 120.0
- link robot11_base_link: mass 120.00000 -> 120.0
- link robot11_link_1: mass 120.00000 -> 120.0
- link robot11_link_2: mass 120.00000 -> 120.0
- link robot11_link_3: mass 120.00000 -> 120.0
- link robot11_link_4: mass 40.00000 -> 40.0
- link robot11_link_5: mass 10.00000 -> 10.0
- link robot11_link_6: mass 5.00000 -> 5.0
- link robot11_xy_cart: mass 120.00000 -> 120.0
- link robot12_base: mass 120.00000 -> 120.0
- link robot12_base_link: mass 120.00000 -> 120.0
- link robot12_link_1: mass 120.00000 -> 120.0
- link robot12_link_2: mass 120.00000 -> 120.0
- link robot12_link_3: mass 120.00000 -> 120.0
- link robot12_link_4: mass 40.00000 -> 40.0
- link robot12_link_5: mass 10.00000 -> 10.0
- link robot12_link_6: mass 5.00000 -> 5.0
- link robot12_xy_cart: mass 120.00000 -> 120.0
- link robot21_base: mass 120.00000 -> 120.0
- link robot21_base_link: mass 120.00000 -> 120.0
- link robot21_link_1: mass 120.00000 -> 120.0
- link robot21_link_2: mass 120.00000 -> 120.0
- link robot21_link_3: mass 120.00000 -> 120.0
- link robot21_link_4: mass 40.00000 -> 40.0
- link robot21_link_5: mass 10.00000 -> 10.0
- link robot21_link_6: mass 5.00000 -> 5.0
- link robot21_xy_cart: mass 120.00000 -> 120.0
- link robot22_base: mass 120.00000 -> 120.0
- link robot22_base_link: mass 120.00000 -> 120.0
- link robot22_link_1: mass 120.00000 -> 120.0
- link robot22_link_2: mass 120.00000 -> 120.0
- link robot22_link_3: mass 120.00000 -> 120.0
- link robot22_link_4: mass 40.00000 -> 40.0
- link robot22_link_5: mass 10.00000 -> 10.0
- link robot22_link_6: mass 5.00000 -> 5.0
- link robot22_xy_cart: mass 120.00000 -> 120.0
Joints:
- joint bridge1_joint_EA_X: axis 1 0 0 -> 1.0 0.0 0.0; limit lower=0.0 upper=37.206 effort=100000 velocity=2.618 -> upper=37.206 effort=100000.0 velocity=2.618; origin xyz=0 0 0 rpy=0 0 0 -> xyz=0.0 0.0 0.0 rpy=0.0 0.0 0.0
- joint bridge2_joint_EA_X: axis 1 0 0 -> 1.0 0.0 0.0; limit lower=2.599 upper=39.805 effort=100000 velocity=2.618 -> lower=2.599 upper=39.805 effort=100000.0 velocity=2.618; origin xyz=0 0 0 rpy=0 0 0 -> xyz=0.0 0.0 0.0 rpy=0.0 0.0 0.0
- joint robot11_joint_0: axis (none) -> 1.0 0.0 0.0; origin xyz=0 0 0 rpy=3.14159265359 0 0.0 -> xyz=0.0 0.0 0.0 rpy=-3.1415926535895866 0.0 0.0
- joint robot11_joint_1: axis 0 0 1 -> 0.0 0.0 1.0; limit lower=-3.14159265359 upper=3.14159265359 effort=100000 velocity=2.618 -> lower=-3.14159265359 upper=3.14159265359 effort=100000.0 velocity=2.618; origin xyz=0 0 0 rpy=0 0 0  -> xyz=0.0 0.0 0.0 rpy=0.0 0.0 0.0
- joint robot11_joint_2: axis 0 1 0 -> 0.0 1.0 0.0; limit lower=-1.57079632679 upper=2.61799387799 effort=100000 velocity=2.618 -> lower=-1.57079632679 upper=2.61799387799 effort=100000.0 velocity=2.618; origin xyz=0.175 0 0.495 rpy=0 0 0  -> xyz=0.175 0.0 0.495 rpy=0.0 0.0 0.0
- joint robot11_joint_3: axis 0 1 0 -> 0.0 1.0 0.0; limit lower=-3.14159265359 upper=1.308996939 effort=100000 velocity=2.618 -> lower=-3.14159265359 upper=1.308996939 effort=100000.0 velocity=2.618; origin xyz=0 0 1.095 rpy=0 0 0  -> xyz=0.0 0.0 1.095 rpy=0.0 0.0 0.0
- joint robot11_joint_4: axis 1 0 0 -> 1.0 0.0 0.0; limit lower=-6.98131700798 upper=6.98131700798 effort=10000 velocity=6.2832 -> lower=-6.98131700798 upper=6.98131700798 effort=10000.0 velocity=6.2832; origin xyz=0.331 0 0.175 rpy=0 0 0  -> xyz=0.331 0.0 0.175 rpy=0.0 0.0 0.0
- joint robot11_joint_5: axis 0 1 0 -> 0.0 1.0 0.0; limit lower=-2.18166 upper=2.18166156499 effort=100000 velocity=6.2832 -> lower=-2.18166 upper=2.18166156499 effort=100000.0 velocity=6.2832; origin xyz=0.939 0 0 rpy=0 0 0  -> xyz=0.939 0.0 0.0 rpy=0.0 0.0 0.0
- joint robot11_joint_6: axis 0 0 1 -> 0.0 0.0 1.0; limit lower=-6.98131700798 upper=6.98131700798 effort=100000 velocity=7.854 -> lower=-6.98131700798 upper=6.98131700798 effort=100000.0 velocity=7.854; origin xyz=0.135 0 0 rpy=0 1.57079632679 0 -> xyz=0.135 0.0 0.0 rpy=0.0 1.57079632679 0.0
- joint robot11_joint_6-tool0: axis (none) -> 1.0 0.0 0.0; origin xyz=0 0 0 rpy=0 0 0 -> xyz=0.0 0.0 0.0 rpy=0.0 0.0 0.0
- joint robot11_joint_EA_Y: axis 0 -1 0 -> 0.0 -1.0 0.0; limit lower=-9.65 upper=0.0 effort=100000 velocity=2.618 -> lower=-9.65 effort=100000.0 velocity=2.618; origin xyz=0 0 0 rpy=0 0 0  -> xyz=0.0 0.0 0.0 rpy=0.0 0.0 0.0
- joint robot11_joint_EA_Z: axis 0 0 -1 -> 0.0 0.0 -1.0; limit lower=-4.915 upper=-1.005 effort=100000 velocity=2.618 -> lower=-4.915 upper=-1.005 effort=100000.0 velocity=2.618; origin xyz=0 0 0 rpy=0 0 0  -> xyz=0.0 0.0 0.0 rpy=0.0 0.0 0.0
- joint robot12_joint_0: axis (none) -> 1.0 0.0 0.0; origin xyz=0 0 0 rpy=3.14159265359 0 0.0 -> xyz=0.0 0.0 0.0 rpy=-3.1415926535895866 0.0 0.0
- joint robot12_joint_1: axis 0 0 1 -> 0.0 0.0 1.0; limit lower=-3.14159265359 upper=3.14159265359 effort=100000 velocity=2.618 -> lower=-3.14159265359 upper=3.14159265359 effort=100000.0 velocity=2.618; origin xyz=0 0 0 rpy=0 0 0  -> xyz=0.0 0.0 0.0 rpy=0.0 0.0 0.0
- joint robot12_joint_2: axis 0 1 0 -> 0.0 1.0 0.0; limit lower=-1.57079632679 upper=2.61799387799 effort=100000 velocity=2.618 -> lower=-1.57079632679 upper=2.61799387799 effort=100000.0 velocity=2.618; origin xyz=0.175 0 0.495 rpy=0 0 0  -> xyz=0.175 0.0 0.495 rpy=0.0 0.0 0.0
- joint robot12_joint_3: axis 0 1 0 -> 0.0 1.0 0.0; limit lower=-3.14159265359 upper=1.308996939 effort=100000 velocity=2.618 -> lower=-3.14159265359 upper=1.308996939 effort=100000.0 velocity=2.618; origin xyz=0 0 1.095 rpy=0 0 0  -> xyz=0.0 0.0 1.095 rpy=0.0 0.0 0.0
- joint robot12_joint_4: axis 1 0 0 -> 1.0 0.0 0.0; limit lower=-6.98131700798 upper=6.98131700798 effort=10000 velocity=6.2832 -> lower=-6.98131700798 upper=6.98131700798 effort=10000.0 velocity=6.2832; origin xyz=0.331 0 0.175 rpy=0 0 0  -> xyz=0.331 0.0 0.175 rpy=0.0 0.0 0.0
- joint robot12_joint_5: axis 0 1 0 -> 0.0 1.0 0.0; limit lower=-2.18166 upper=2.18166156499 effort=100000 velocity=6.2832 -> lower=-2.18166 upper=2.18166156499 effort=100000.0 velocity=6.2832; origin xyz=0.939 0 0 rpy=0 0 0  -> xyz=0.939 0.0 0.0 rpy=0.0 0.0 0.0
- joint robot12_joint_6: axis 0 0 1 -> 0.0 0.0 1.0; limit lower=-6.98131700798 upper=6.98131700798 effort=100000 velocity=7.854 -> lower=-6.98131700798 upper=6.98131700798 effort=100000.0 velocity=7.854; origin xyz=0.135 0 0 rpy=0 1.57079632679 0 -> xyz=0.135 0.0 0.0 rpy=0.0 1.57079632679 0.0
- joint robot12_joint_6-tool0: axis (none) -> 1.0 0.0 0.0; origin xyz=0 0 0 rpy=0 0 0 -> xyz=0.0 0.0 0.0 rpy=0.0 0.0 0.0
- joint robot12_joint_EA_Y: axis 0 -1 0 -> 0.0 -1.0 0.0; limit lower=-12.237 upper=-2.587 effort=100000 velocity=2.618 -> lower=-12.237 upper=-2.587 effort=100000.0 velocity=2.618; origin xyz=0 0 0 rpy=0 0 0  -> xyz=0.0 0.0 0.0 rpy=0.0 0.0 0.0
- joint robot12_joint_EA_Z: axis 0 0 -1 -> 0.0 0.0 -1.0; limit lower=-4.915 upper=-1.005 effort=100000 velocity=2.618 -> lower=-4.915 upper=-1.005 effort=100000.0 velocity=2.618; origin xyz=0 0 0 rpy=0 0 0  -> xyz=0.0 0.0 0.0 rpy=0.0 0.0 0.0
- joint robot21_joint_0: axis (none) -> 1.0 0.0 0.0; origin xyz=0 0 0 rpy=3.14159265359 0 3.14159265359 -> xyz=0.0 0.0 0.0 rpy=-3.1415926535895866 0.0 -3.1415926535895866
- joint robot21_joint_1: axis 0 0 1 -> 0.0 0.0 1.0; limit lower=-3.14159265359 upper=3.14159265359 effort=100000 velocity=2.618 -> lower=-3.14159265359 upper=3.14159265359 effort=100000.0 velocity=2.618; origin xyz=0 0 0 rpy=0 0 0  -> xyz=0.0 0.0 0.0 rpy=0.0 0.0 0.0
- joint robot21_joint_2: axis 0 1 0 -> 0.0 1.0 0.0; limit lower=-1.57079632679 upper=2.61799387799 effort=100000 velocity=2.618 -> lower=-1.57079632679 upper=2.61799387799 effort=100000.0 velocity=2.618; origin xyz=0.175 0 0.495 rpy=0 0 0  -> xyz=0.175 0.0 0.495 rpy=0.0 0.0 0.0
- joint robot21_joint_3: axis 0 1 0 -> 0.0 1.0 0.0; limit lower=-3.14159265359 upper=1.308996939 effort=100000 velocity=2.618 -> lower=-3.14159265359 upper=1.308996939 effort=100000.0 velocity=2.618; origin xyz=0 0 1.095 rpy=0 0 0  -> xyz=0.0 0.0 1.095 rpy=0.0 0.0 0.0
- joint robot21_joint_4: axis 1 0 0 -> 1.0 0.0 0.0; limit lower=-6.98131700798 upper=6.98131700798 effort=10000 velocity=6.2832 -> lower=-6.98131700798 upper=6.98131700798 effort=10000.0 velocity=6.2832; origin xyz=0.331 0 0.175 rpy=0 0 0  -> xyz=0.331 0.0 0.175 rpy=0.0 0.0 0.0
- joint robot21_joint_5: axis 0 1 0 -> 0.0 1.0 0.0; limit lower=-2.18166 upper=2.18166156499 effort=100000 velocity=6.2832 -> lower=-2.18166 upper=2.18166156499 effort=100000.0 velocity=6.2832; origin xyz=0.939 0 0 rpy=0 0 0  -> xyz=0.939 0.0 0.0 rpy=0.0 0.0 0.0
- joint robot21_joint_6: axis 0 0 1 -> 0.0 0.0 1.0; limit lower=-6.98131700798 upper=6.98131700798 effort=100000 velocity=7.854 -> lower=-6.98131700798 upper=6.98131700798 effort=100000.0 velocity=7.854; origin xyz=0.135 0 0 rpy=0 1.57079632679 0 -> xyz=0.135 0.0 0.0 rpy=0.0 1.57079632679 0.0
- joint robot21_joint_6-tool0: axis (none) -> 1.0 0.0 0.0; origin xyz=0 0 0 rpy=0 0 0 -> xyz=0.0 0.0 0.0 rpy=0.0 0.0 0.0
- joint robot21_joint_EA_Y: axis 0 -1 0 -> 0.0 -1.0 0.0; limit lower=-9.65 upper=0.0 effort=100000 velocity=2.618 -> lower=-9.65 effort=100000.0 velocity=2.618; origin xyz=0 0 0 rpy=0 0 0  -> xyz=0.0 0.0 0.0 rpy=0.0 0.0 0.0
- joint robot21_joint_EA_Z: axis 0 0 -1 -> 0.0 0.0 -1.0; limit lower=-4.915 upper=-1.005 effort=100000 velocity=2.618 -> lower=-4.915 upper=-1.005 effort=100000.0 velocity=2.618; origin xyz=0 0 0 rpy=0 0 0  -> xyz=0.0 0.0 0.0 rpy=0.0 0.0 0.0
- joint robot22_joint_0: axis (none) -> 1.0 0.0 0.0; origin xyz=0 0 0 rpy=3.14159265359 0 3.14159265359 -> xyz=0.0 0.0 0.0 rpy=-3.1415926535895866 0.0 -3.1415926535895866
- joint robot22_joint_1: axis 0 0 1 -> 0.0 0.0 1.0; limit lower=-3.14159265359 upper=3.14159265359 effort=100000 velocity=2.618 -> lower=-3.14159265359 upper=3.14159265359 effort=100000.0 velocity=2.618; origin xyz=0 0 0 rpy=0 0 0  -> xyz=0.0 0.0 0.0 rpy=0.0 0.0 0.0
- joint robot22_joint_2: axis 0 1 0 -> 0.0 1.0 0.0; limit lower=-1.57079632679 upper=2.61799387799 effort=100000 velocity=2.618 -> lower=-1.57079632679 upper=2.61799387799 effort=100000.0 velocity=2.618; origin xyz=0.175 0 0.495 rpy=0 0 0  -> xyz=0.175 0.0 0.495 rpy=0.0 0.0 0.0
- joint robot22_joint_3: axis 0 1 0 -> 0.0 1.0 0.0; limit lower=-3.14159265359 upper=1.308996939 effort=100000 velocity=2.618 -> lower=-3.14159265359 upper=1.308996939 effort=100000.0 velocity=2.618; origin xyz=0 0 1.095 rpy=0 0 0  -> xyz=0.0 0.0 1.095 rpy=0.0 0.0 0.0
- joint robot22_joint_4: axis 1 0 0 -> 1.0 0.0 0.0; limit lower=-6.98131700798 upper=6.98131700798 effort=10000 velocity=6.2832 -> lower=-6.98131700798 upper=6.98131700798 effort=10000.0 velocity=6.2832; origin xyz=0.331 0 0.175 rpy=0 0 0  -> xyz=0.331 0.0 0.175 rpy=0.0 0.0 0.0
- joint robot22_joint_5: axis 0 1 0 -> 0.0 1.0 0.0; limit lower=-2.18166 upper=2.18166156499 effort=100000 velocity=6.2832 -> lower=-2.18166 upper=2.18166156499 effort=100000.0 velocity=6.2832; origin xyz=0.939 0 0 rpy=0 0 0  -> xyz=0.939 0.0 0.0 rpy=0.0 0.0 0.0
- joint robot22_joint_6: axis 0 0 1 -> 0.0 0.0 1.0; limit lower=-6.98131700798 upper=6.98131700798 effort=100000 velocity=7.854 -> lower=-6.98131700798 upper=6.98131700798 effort=100000.0 velocity=7.854; origin xyz=0.135 0 0 rpy=0 1.57079632679 0 -> xyz=0.135 0.0 0.0 rpy=0.0 1.57079632679 0.0
- joint robot22_joint_6-tool0: axis (none) -> 1.0 0.0 0.0; origin xyz=0 0 0 rpy=0 0 0 -> xyz=0.0 0.0 0.0 rpy=0.0 0.0 0.0
- joint robot22_joint_EA_Y: axis 0 -1 0 -> 0.0 -1.0 0.0; limit lower=-12.237 upper=-2.587 effort=100000 velocity=2.618 -> lower=-12.237 upper=-2.587 effort=100000.0 velocity=2.618; origin xyz=0 0 0 rpy=0 0 0  -> xyz=0.0 0.0 0.0 rpy=0.0 0.0 0.0
- joint robot22_joint_EA_Z: axis 0 0 -1 -> 0.0 0.0 -1.0; limit lower=-4.915 upper=-1.005 effort=100000 velocity=2.618 -> lower=-4.915 upper=-1.005 effort=100000.0 velocity=2.618; origin xyz=0 0 0 rpy=0 0 0  -> xyz=0.0 0.0 0.0 rpy=0.0 0.0 0.0
- joint world_joint: axis (none) -> 1.0 0.0 0.0
