Commit message: Refresh bundled analytical robot cells

File: src/compas_fab/data/robot_library/ur10e_robot/urdf/robot_description.urdf (robot description, URDF)
Before this commit: robot ur10e_robot, 11 links, 10 joints
Links:
- added link ft_frame
- link base_link_inertia: geometry collision mesh filename=package://ur_description/meshes/ur10e/collision/base.stl; visual mesh filename=package://ur_description/meshes/ur10e/visual/base.dae
- link forearm_link: mass 3.87 -> 3.989; geometry collision mesh filename=package://ur_description/meshes/ur10e/collision/forearm.stl; visual mesh filename=package://ur_description/meshes/ur10e/visual/forearm.dae
- link shoulder_link: mass 7.778 -> 7.369; geometry collision mesh filename=package://ur_description/meshes/ur10e/collision/shoulder.stl; visual mesh filename=package://ur_description/meshes/ur10e/visual/shoulder.dae
- link upper_arm_link: mass 12.93 -> 13.051; geometry collision mesh filename=package://ur_description/meshes/ur10e/collision/upperarm.stl; visual mesh filename=package://ur_description/meshes/ur10e/visual/upperarm.dae
- link wrist_1_link: mass 1.96 -> 2.1; geometry collision mesh filename=package://ur_description/meshes/ur10e/collision/wrist1.stl; visual mesh filename=package://ur_description/meshes/ur10e/visual/wrist1.dae
- link wrist_2_link: mass 1.96 -> 1.98; geometry collision mesh filename=package://ur_description/meshes/ur10e/collision/wrist2.stl; visual mesh filename=package://ur_description/meshes/ur10e/visual/wrist2.dae
- link wrist_3_link: mass 0.202 -> 0.615; geometry collision mesh filename=package://ur_description/meshes/ur10e/collision/wrist3.stl; visual mesh filename=package://ur_description/meshes/ur10e/visual/wrist3.dae
Joints:
- added joint wrist_3_link-ft_frame: type fixed, parent wrist_3_link, child ft_frame, origin xyz=0 0 0 rpy=3.141592653589793 0 0
- joint base_link-base_fixed_joint: axis 1.0 0.0 0.0 -> (none); origin xyz=0.0 0.0 0.0 rpy=0.0 0.0 3.141592653589793 -> xyz=0 0 0 rpy=0 0 3.141592653589793
- joint base_link-base_link_inertia: axis 1.0 0.0 0.0 -> (none); origin xyz=0.0 0.0 0.0 rpy=0.0 0.0 3.141592653589793 -> xyz=0 0 0 rpy=0 0 3.141592653589793
- joint elbow_joint: axis 0.0 0.0 1.0 -> 0 0 1; origin xyz=-0.6127 0.0 0.0 rpy=0.0 0.0 0.0 -> xyz=-0.6127 0 0 rpy=0 0 0
- joint flange-tool0: axis 1.0 0.0 0.0 -> (none); origin xyz=0.0 0.0 0.0 rpy=1.5707963267948966 0.0 1.5707963267948966 -> xyz=0 0 0 rpy=1.5707963267948966 0 1.5707963267948966
- joint shoulder_lift_joint: axis 0.0 0.0 1.0 -> 0 0 1; origin xyz=0.0 0.0 0.0 rpy=1.570796327 0.0 0.0 -> xyz=0 0 0 rpy=1.570796327 0 0
- joint shoulder_pan_joint: axis 0.0 0.0 1.0 -> 0 0 1; origin xyz=0.0 0.0 0.1807 rpy=0.0 0.0 0.0 -> xyz=0 0 0.1807 rpy=0 0 0
- joint wrist_1_joint: axis 0.0 0.0 1.0 -> 0 0 1; limit lower=-6.283185307179586 upper=6.283185307179586 effort=56.0 velocity=3.141592653589793 -> lower=-6.283185307179586 upper=6.283185307179586 effort=54.0 velocity=3.141592653589793; origin xyz=-0.57155 0.0 0.17415 rpy=0.0 0.0 0.0 -> xyz=-0.57155 0 0.17415 rpy=0 0 0
- joint wrist_2_joint: axis 0.0 0.0 1.0 -> 0 0 1; limit lower=-6.283185307179586 upper=6.283185307179586 effort=56.0 velocity=3.141592653589793 -> lower=-6.283185307179586 upper=6.283185307179586 effort=54.0 velocity=3.141592653589793; origin xyz=0.0 -0.11985 -2.458164590756244e-11 rpy=1.570796327 0.0 0.0 -> xyz=0 -0.11985 -2.458164590756244e-11 rpy=1.570796327 0 0
- joint wrist_3-flange: axis 1.0 0.0 0.0 -> (none); origin xyz=0.0 0.0 0.0 rpy=-1.5707963267948966 -1.5707963267948966 0.0 -> xyz=0 0 0 rpy=0 -1.5707963267948966 -1.5707963267948966
- joint wrist_3_joint: axis 0.0 0.0 1.0 -> 0 0 1; limit lower=-6.283185307179586 upper=6.283185307179586 effort=56.0 velocity=3.141592653589793 -> lower=-6.283185307179586 upper=6.283185307179586 effort=54.0 velocity=3.141592653589793; origin xyz=0.0 0.11655 -2.390480459346185e-11 rpy=-1.5707963270000003 1.2246467991473532e-16 -1.2246467991473532e-16 -> xyz=0 0.11655 -2.390480459346185e-11 rpy=1.570796326589793 3.141592653589793 3.141592653589793

File: src/compas_fab/data/robot_library/ur5_robot/urdf/robot_description.urdf (robot description, URDF)
Before this commit: robot ur5_robot, 11 links, 10 joints
Links:
- added link ft_frame
- link base_link_inertia: geometry collision mesh filename=package://ur_description/meshes/ur5/collision/base.stl; visual mesh filename=package://ur_description/meshes/ur5/visual/base.dae
- link forearm_link: mass 2.275 -> 2.33; geometry collision mesh filename=package://ur_description/meshes/ur5/collision/forearm.stl; visual mesh filename=package://ur_description/meshes/ur5/visual/forearm.dae
- link shoulder_link: geometry collision mesh filename=package://ur_description/meshes/ur5/collision/shoulder.stl; visual mesh filename=package://ur_description/meshes/ur5/visual/shoulder.dae
- link upper_arm_link: geometry collision mesh filename=package://ur_description/meshes/ur5/collision/upperarm.stl; visual mesh filename=package://ur_description/meshes/ur5/visual/upperarm.dae
- link wrist_1_link: geometry collision mesh filename=package://ur_description/meshes/ur5/collision/wrist1.stl; visual mesh filename=package://ur_description/meshes/ur5/visual/wrist1.dae
- link wrist_2_link: geometry collision mesh filename=package://ur_description/meshes/ur5/collision/wrist2.stl; visual mesh filename=package://ur_description/meshes/ur5/visual/wrist2.dae
- link wrist_3_link: geometry collision mesh filename=package://ur_description/meshes/ur5/collision/wrist3.stl; visual mesh filename=package://ur_description/meshes/ur5/visual/wrist3.dae
Joints:
- added joint wrist_3_link-ft_frame: type fixed, parent wrist_3_link, child ft_frame, origin xyz=0 0 0 rpy=3.141592653589793 0 0
- joint base_link-base_fixed_joint: axis 1.0 0.0 0.0 -> (none); origin xyz=0.0 0.0 0.0 rpy=0.0 0.0 3.141592653589793 -> xyz=0 0 0 rpy=0 0 3.141592653589793
- joint base_link-base_link_inertia: axis 1.0 0.0 0.0 -> (none); origin xyz=0.0 0.0 0.0 rpy=0.0 0.0 3.141592653589793 -> xyz=0 0 0 rpy=0 0 3.141592653589793
- joint elbow_joint: axis 0.0 0.0 1.0 -> 0 0 1; origin xyz=-0.425 0.0 0.0 rpy=0.0 0.0 0.0 -> xyz=-0.425 0 0 rpy=0 0 0
- joint flange-tool0: axis 1.0 0.0 0.0 -> (none); origin xyz=0.0 0.0 0.0 rpy=1.5707963267948966 0.0 1.5707963267948966 -> xyz=0 0 0 rpy=1.5707963267948966 0 1.5707963267948966
- joint shoulder_lift_joint: axis 0.0 0.0 1.0 -> 0 0 1; origin xyz=0.0 0.0 0.0 rpy=1.570796327 0.0 0.0 -> xyz=0 0 0 rpy=1.570796327 0 0
- joint shoulder_pan_joint: axis 0.0 0.0 1.0 -> 0 0 1; origin xyz=0.0 0.0 0.089159 rpy=0.0 0.0 0.0 -> xyz=0 0 0.089159 rpy=0 0 0
- joint wrist_1_joint: axis 0.0 0.0 1.0 -> 0 0 1; origin xyz=-0.39225 0.0 0.10915 rpy=0.0 0.0 0.0 -> xyz=-0.39225 0 0.10915 rpy=0 0 0
- joint wrist_2_joint: axis 0.0 0.0 1.0 -> 0 0 1; origin xyz=0.0 -0.09465 -1.941303950897609e-11 rpy=1.570796327 0.0 0.0 -> xyz=0 -0.09465 -1.941303950897609e-11 rpy=1.570796327 0 0
- joint wrist_3-flange: axis 1.0 0.0 0.0 -> (none); origin xyz=0.0 0.0 0.0 rpy=-1.5707963267948966 -1.5707963267948966 0.0 -> xyz=0 0 0 rpy=0 -1.5707963267948966 -1.5707963267948966
- joint wrist_3_joint: axis 0.0 0.0 1.0 -> 0 0 1; origin xyz=0.0 0.0823 -1.688001216681175e-11 rpy=-1.5707963270000003 1.2246467991473532e-16 -1.2246467991473532e-16 -> xyz=0 0.0823 -1.688001216681175e-11 rpy=1.570796326589793 3.141592653589793 3.141592653589793
